File: main/pcb_challenge_final.kicad_pcb (KiCad board)
At the start: 2 copper layers, 164 parts, among them J4 Conn_01x04_Pin, J5 Conn_01x04_Pin, Q15 Q_Dual_NPN_PNP_B1E2B2C2E1C1, Q16 Q_Dual_NPN_PNP_B1E2B2C2E1C1, Q17 Q_Dual_NPN_PNP_B1E2B2C2E1C1, Q18 Q_Dual_NPN_PNP_B1E2B2C2E1C1, Q19 Q_Dual_NPN_PNP_B1E2B2C2E1C1, Q20 Q_Dual_NPN_PNP_B1E2B2C2E1C1, Q21 Q_Dual_NPN_PNP_B1E2B2C2E1C1, Q22 Q_Dual_NPN_PNP_B1E2B2C2E1C1, Q23 Q_Dual_NPN_PNP_B1E2B2C2E1C1, Q24 Q_Dual_NPN_PNP_B1E2B2C2E1C1, Q25 Q_Dual_NPN_PNP_B1E2B2C2E1C1, Q26 Q_Dual_NPN_PNP_B1E2B2C2E1C1, Q27 Q_Dual_NPN_PNP_B1E2B2C2E1C1, Q28 Q_Dual_NPN_PNP_B1E2B2C2E1C1, Q29 Q_Dual_NPN_PNP_B1E2B2C2E1C1, SW1 SW_Push, SW2 SW_Push, SW3 SW_Push, U1 74AUP1G80, U10 NMUX1308BQ, U11 NMUX1308BQ, U12 NMUX1308BQ, U13 NMUX1308BQ, U14 NMUX1308BQ, U15 NMUX1308BQ, U16 NMUX1308BQ, U17 74AUP1G80, U18 74AHC1G86, U19 74AUP1G80, U20 74AUP1G80, U21 74LV1T08GV, U22 CD74HC283M96, U23 74LV1T08GV, U24 74LVC1GU04DRL, U25 ESP32-S3-MINI-1, U26 74LVC1GU04DRL, U27 74LV1T08GV, U28 CD74HC283M96, U29 NMUX1308BQ, U3 74AHC1G86, U30 NMUX1308BQ, U31 NMUX1308BQ, U32 NMUX1308BQ, U33 74AUP1G80, U34 74AUP1G80, U35 NMUX1308BQ, U36 NMUX1308BQ, U37 74AUP1G80, U38 74AUP1G80, U39 NMUX1308BQ, U4 74AUP1G80, U40 NMUX1308BQ, U41 NMUX1308BQ, U42 NMUX1308BQ, U43 NMUX1308BQ, U44 NMUX1308BQ, U45 74AUP1G80, U46 74AUP1G80, U47 74AUP1G80, U48 74AUP1G80, U49 74AUP1G80, U5 74AUP1G80, U50 74AUP1G80, U51 74LV1T08GV, U52 74AHC1G86, U53 74LVC1GU04DRL, U54 74LVC1GU04DRL, U55 74AHC1G86, U56 74AHC1G86, U57 74LVC1GU04DRL, U58 74LVC1GU04DRL, U59 74LV1T08GV, U6 74AUP1G80, U60 74AHC1G86, U61 74LVC1GU04DRL, U62 74LV1T08GV, U63 74LV1T08GV, U64 NMUX1308BQ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

Commit message: chore: remove duplicate SW2
Parts:
- SW2: value SW_Push -> SW_MEC_5G; footprint Button_Switch_SMD:SW_DIP_SPSTx01_Slide_6.7x4.1mm_W8.61mm_P2.54mm_LowProfile -> Button_Switch_SMD:SW_SPST_CK_RS282G05A3
- moved SW2 106.6 mm to (114.5, 111.0)
Connections:
- C9 pad 1: rst -> NRST
- SW2 pad 2: rst -> GND

Commit message: feat: routed OUTREG and EMPTY subcircuits
Parts:
- moved Y2 163.9 mm to (37.2, 25.5)
- moved U6 147.9 mm to (65.3, 27.0)
- moved U7 146.5 mm to (67.2, 21.3)
- moved U8 146.5 mm to (67.2, 23.9)
- moved Q15 145.3 mm to (40.8, 53.2)
- moved Q28 145.3 mm to (41.0, 49.0)
- moved Q29 145.3 mm to (41.0, 51.2)
- moved R7 145.2 mm to (31.7, 26.5)
- moved Q17 140.5 mm to (40.7, 45.8)
- moved U22 136.1 mm to (95.9, 28.9)
- moved U45 130.8 mm to (132.0, 19.3)
- moved U46 130.8 mm to (132.0, 21.9)
- moved U47 130.8 mm to (132.0, 24.5)
- moved U48 130.8 mm to (134.7, 16.7)
- moved U49 130.8 mm to (134.7, 19.3)
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Routing:
- net IO6: track 0.00 -> 33.6 mm, vias 0 -> 5
- net r_en: track 0.00 -> 24.3 mm, vias 0 -> 5
- net IO8: track 0.00 -> 24.2 mm
- net out_1: track 0.00 -> 20.1 mm
- net out_2: track 0.00 -> 14.7 mm
- net GND: track 0.00 -> 13.3 mm, vias 0 -> 3
- net Net-(U28-A3): track 0.00 -> 10.5 mm, vias 0 -> 2
- net wc3: track 0.00 -> 10.4 mm
- net out_3: track 0.00 -> 9.19 mm
- net Net-(U55-Pad4): track 0.00 -> 7.95 mm
- net wc1: track 0.00 -> 7.29 mm
- net Net-(U59-B): track 0.00 -> 5.33 mm
- net Net-(U59-Y): track 0.00 -> 4.71 mm
- net Net-(U21-B): track 0.00 -> 4.33 mm
- net out_4: track 0.00 -> 3.85 mm
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- added copper zone on In2.Cu, net +3.3V
- added copper zone on In1.Cu, net GND
Other:
- copper layers 2 -> 4

Commit message: chore: clean up RPTR subcircuit
Parts:
- moved U14 9.97 mm to (200.5, 61.4), turned to 0 degrees
- moved U19 9.34 mm to (199.9, 64.1), turned to 0 degrees
- moved R44 8.85 mm to (211.7, 61.6), turned to 180 degrees
- moved U17 6.55 mm to (208.8, 60.2), turned to 180 degrees
- moved U72 5.98 mm to (127.2, 130.0)
- moved R62 5.98 mm to (129.4, 129.7)
- moved Q22 5.38 mm to (197.6, 62.9), turned to 180 degrees
- moved R45 5.30 mm to (197.4, 65.5)
- moved U15 5.22 mm to (200.2, 66.2), turned to 0 degrees
- moved U66 5.14 mm to (127.1, 126.7)
- moved Q24 5.14 mm to (129.1, 126.6)
- moved Q21 4.75 mm to (212.3, 63.3), turned to 0 degrees
- moved R64 4.21 mm to (129.4, 123.2)
- moved U71 4.21 mm to (127.2, 123.5)
- moved Q25 3.40 mm to (129.1, 120.2)
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Routing:
- net GND: track 13.3 -> 61.9 mm, vias 3 -> 29
- net +3.3V: track 0.00 -> 46.2 mm, vias 0 -> 27
- net out_1: track 20.1 -> 0.00 mm
- net out_2: track 14.7 -> 0.00 mm
- net IO6: track 33.6 -> 47.5 mm, vias 5 -> 6
- net R_en: track 0.00 -> 12.3 mm
- net rst: track 3.05 -> 13.5 mm
- net IO8: track 24.2 -> 34.4 mm
- net out_3: track 9.19 -> 0.00 mm
- net Net-(U55-Pad4): track 7.95 -> 0.00 mm
- net wc2: track 0.00 -> 7.45 mm
- net r_en: track 24.3 -> 31.8 mm, vias 5 -> 0
- net Net-(U28-A3): track 10.5 -> 17.1 mm, vias 2 -> 5
- net clk: track 3.28 -> 9.64 mm, vias 3 -> 2
- net Net-(U64-Out): track 0.00 -> 5.74 mm
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
Commit message: feat: routed middle blocks
Parts:
- moved U17 120.7 mm to (110.5, 130.2), turned to -90 degrees
- moved R47 119.6 mm to (110.6, 135.4), turned to -90 degrees
- moved R44 119.5 mm to (111.9, 127.3), turned to -90 degrees
- moved U14 117.7 mm to (111.6, 138.5), turned to 90 degrees
- moved Q21 117.4 mm to (113.5, 126.7), turned to 90 degrees
- moved Q22 115.3 mm to (113.2, 141.4), turned to -90 degrees
- moved U16 114.6 mm to (115.4, 127.3), turned to -90 degrees
- moved U19 113.8 mm to (114.4, 139.1), turned to 90 degrees
- moved R45 111.7 mm to (115.7, 141.6), turned to 180 degrees
- moved U28 111.3 mm to (116.7, 133.2), turned to 90 degrees
- moved U15 110.9 mm to (116.4, 138.8), turned to 90 degrees
- moved U20 106.8 mm to (119.3, 139.3), turned to -90 degrees
- moved Q23 104.5 mm to (120.8, 140.1), turned to -90 degrees
- moved R34 104.1 mm to (121.3, 137.8), turned to 180 degrees
- moved R46 102.5 mm to (122.3, 140.2), turned to -90 degrees
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Routing:
- net GND: track 61.9 -> 132.1 mm, vias 29 -> 48
- net +3.3V: track 46.2 -> 106.4 mm, vias 27 -> 45
- net rst: track 13.5 -> 48.5 mm
- net clk: track 9.64 -> 38.1 mm, vias 2 -> 8
- net USB_D-: track 0.00 -> 13.5 mm
- net USB_D+: track 0.00 -> 12.5 mm, vias 0 -> 2
- net Net-(U31-Y1): track 0.00 -> 10.2 mm, vias 0 -> 2
- net IO6: track 47.5 -> 54.2 mm, vias 6 -> 12
- net Net-(U42-Y0): track 0.00 -> 6.60 mm
- net Net-(U43-Y0): track 0.00 -> 6.58 mm
- net Net-(U44-Y0): track 0.00 -> 6.39 mm
- net r_en: track 31.8 -> 25.9 mm
- net Net-(U32-Y0): track 0.00 -> 3.70 mm
- net Net-(U30-Y0): track 0.00 -> 3.67 mm
- net Net-(U36-Y0): track 0.00 -> 3.48 mm
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
Commit message: chore: add capacitors to USB polarity headers
Parts:
- moved SW3 39.6 mm to (147.7, 138.4), turned to -90 degrees
- moved R1 30.9 mm to (140.3, 140.3), turned to 180 degrees
- moved C8 28.5 mm to (140.2, 139.4)
- moved C7 27.5 mm to (140.2, 138.7)
- moved C6 8.57 mm to (140.1, 122.3), turned to -90 degrees
- moved SW1 6.67 mm to (129.0, 160.4)
- moved C5 5.28 mm to (140.1, 124.4), turned to 90 degrees
Routing:
- net Net-(U25-EN): track 0.00 -> 31.1 mm
- net GND: track 132.1 -> 134.3 mm, vias 48 -> 49
- net USB_D+: track 12.5 -> 14.4 mm, vias 2 -> 3
- net USB_D-: track 13.5 -> 14.4 mm

Commit message: chore: route longer connections
Parts:
- moved U7 122.0 mm to (105.2, 137.3)
- moved R25 120.2 mm to (104.2, 146.1), turned to 90 degrees
- moved U8 115.7 mm to (109.5, 131.6)
- moved R33 115.4 mm to (105.9, 144.9), turned to 90 degrees
- moved U6 115.0 mm to (106.0, 134.6)
- moved U22 114.4 mm to (111.0, 142.3)
- moved Q18 113.0 mm to (104.6, 132.1), turned to 180 degrees
- moved Q20 112.7 mm to (102.7, 136.7), turned to -90 degrees
- moved Q19 111.3 mm to (106.7, 132.0), turned to 90 degrees
- moved R36 110.2 mm to (102.4, 140.2), turned to 90 degrees
- moved U12 105.0 mm to (105.0, 140.8), turned to -90 degrees
- moved U11 103.7 mm to (109.5, 134.7), turned to 180 degrees
- moved Y2 99.3 mm to (67.2, 131.6), turned to -90 degrees
- moved U13 98.0 mm to (113.6, 134.3), turned to -90 degrees
- moved R38 96.7 mm to (107.6, 129.4), turned to 180 degrees
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Routing:
- net clk: track 38.1 -> 134.3 mm, vias 8 -> 15
- net rw1: track 0.00 -> 88.0 mm, vias 0 -> 9
- net IO8: track 34.4 -> 121.1 mm, vias 0 -> 16
- net IO6: track 54.2 -> 138.7 mm, vias 12 -> 20
- net rst: track 48.5 -> 127.4 mm, vias 3 -> 12
- net rw3: track 0.00 -> 76.0 mm, vias 0 -> 10
- net wc2: track 7.45 -> 76.8 mm, vias 0 -> 8
- net rc1: track 0.00 -> 69.0 mm, vias 0 -> 15
- net out_2: track 0.00 -> 68.1 mm, vias 0 -> 10
- net GND: track 134.3 -> 200.6 mm, vias 49 -> 109
- net rc2: track 0.00 -> 65.8 mm, vias 0 -> 7
- net rw2: track 0.00 -> 64.6 mm, vias 0 -> 4
- net out_3: track 0.00 -> 61.0 mm, vias 0 -> 10
- net wc1: track 11.4 -> 72.0 mm, vias 2 -> 6
- net b3: track 0.00 -> 54.0 mm, vias 0 -> 1
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
Commit message: chore: move connectors closer left
Parts:
- moved C9 45.7 mm to (119.0, 143.1)
- moved SW2 45.7 mm to (125.3, 143.4)
- moved R21 15.2 mm to (105.1, 112.5)
- moved R23 15.2 mm to (103.6, 112.5)
- moved R27 15.2 mm to (108.1, 112.5)
- moved R29 15.2 mm to (106.6, 112.5)
- moved R31 15.2 mm to (97.6, 112.5)
- moved R41 15.2 mm to (102.1, 112.5)
- moved R42 15.2 mm to (100.6, 112.5)
- moved R43 15.2 mm to (99.1, 112.5)
- moved Q16 5.91 mm to (75.5, 117.7)
- moved Q28 5.91 mm to (65.1, 129.9)
- moved R26 5.91 mm to (65.1, 132.4)
- moved R30 5.91 mm to (61.9, 132.4)
- moved R32 5.91 mm to (75.5, 114.5)
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Routing:
- net Net-(U25-GND-Pad2): track 0.00 -> 55.3 mm
- net rst: track 127.4 -> 138.3 mm
- net IO8: track 121.1 -> 131.8 mm, vias 16 -> 18
- net Net-(U25-IO0): track 34.4 -> 25.5 mm
- net rw3: track 76.0 -> 69.0 mm, vias 10 -> 12
- net wc2: track 76.8 -> 69.9 mm
- net wc3: track 42.8 -> 36.9 mm
- net GND: track 200.6 -> 194.8 mm, vias 109 -> 101
- net R_en: track 65.0 -> 59.2 mm
- net clk: track 134.3 -> 128.5 mm
- net b1: track 42.4 -> 36.6 mm
- net b3: track 54.0 -> 48.3 mm
- net b4: track 53.8 -> 48.1 mm
- net b2: track 45.9 -> 40.2 mm
- net rw1: track 88.0 -> 83.0 mm, vias 9 -> 8
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Other:
- board outline added: 100.3 x 44.7 mm

Commit message: chore: rerouting
Parts:
- moved J5 39.6 mm to (75.8, 143.5), turned to 90 degrees
- moved J4 19.6 mm to (63.2, 138.5), turned to 90 degrees
Routing:
- net en: track 42.5 -> 18.9 mm, vias 0 -> 3
- net rst: track 138.3 -> 154.8 mm, vias 12 -> 13
- net b3: track 48.3 -> 35.2 mm, vias 1 -> 0
- net b4: track 48.1 -> 37.7 mm, vias 4 -> 3
- net b2: track 40.2 -> 32.5 mm, vias 1 -> 0
- net b1: track 36.6 -> 29.5 mm, vias 2 -> 0
- net ???: track 28.6 -> 21.6 mm, vias 0 -> 3
- net Net-(U25-IO0): track 25.5 -> 31.3 mm
- net clk: track 128.5 -> 125.4 mm, vias 15 -> 16
- net GND: track 194.8 -> 197.3 mm, vias 101 -> 102
Other:
- board size 100.3 x 44.7 mm -> 89.4 x 44.8 mm
